Commit message: [OK] panda, dual_panda, [doing] timda

File: manipulability_metrics_examples/urdf/dual_panda.urdf.xacro (robot description, xacro)
@@ -1,10 +1,14 @@
 <?xml version="1.0" encoding="utf-8"?>
 <robot xmlns:xacro="http://www.ros.org/wiki/xacro" name="dual_panda">
-  <xacro:include filename="$(find franka_description)/robots/panda_arm.xacro"/>
-  <xacro:include filename="$(find franka_description)/robots/hand.xacro"/>
-  <link name="base_link" />
-  <xacro:panda_arm arm_id="left_panda" connected_to="base_link" xyz="0 0.25 0" />
-  <xacro:hand ns="left_panda" rpy="0 0 ${-pi/4}" connected_to="left_panda_link8"/>
-  <xacro:panda_arm arm_id="right_panda" connected_to="base_link" xyz="0 -0.25 0" />
-  <xacro:hand ns="right_panda" rpy="0 0 ${-pi/4}" connected_to="right_panda_link8"/>
+  <xacro:arg name="arm_id_1" default="left_panda" />
+  <xacro:arg name="arm_id_2" default="right_panda" />
+  <xacro:include filename="$(find franka_description)/robots/common/franka_arm.xacro"/>
+  <xacro:include filename="$(find franka_description)/robots/common/franka_hand.xacro"/>
+  <link name="base"/>
+  <!-- Panda left arm with hand -->
+  <xacro:franka_arm arm_id="$(arg arm_id_1)" connected_to="base"  xyz="0 0.25 0" safety_distance="0.03" joint_limits="${xacro.load_yaml('$(find franka_description)/robots/panda/joint_limits.yaml')}"/>
+  <xacro:franka_hand arm_id="$(arg arm_id_1)" rpy="0 0 ${-pi/4}" connected_to="$(arg arm_id_1)_link8" safety_distance="0.03"/>
+  <!-- Panda right arm with hand -->
+  <xacro:franka_arm arm_id="$(arg arm_id_2)" connected_to="base"  xyz="0 -0.25 0" safety_distance="0.03" joint_limits="${xacro.load_yaml('$(find franka_description)/robots/panda/joint_limits.yaml')}"/>
+  <xacro:franka_hand arm_id="$(arg arm_id_2)" rpy="0 0 ${-pi/4}" connected_to="$(arg arm_id_2)_link8" safety_distance="0.03"/>
 </robot>

File: manipulability_metrics_examples/urdf/panda.urdf.xacro (robot description, xacro)
@@ -1,8 +1,11 @@
 <?xml version="1.0" encoding="utf-8"?>
 <robot xmlns:xacro="http://www.ros.org/wiki/xacro" name="panda">
-  <xacro:include filename="$(find franka_description)/robots/panda_arm.xacro"/>
-  <xacro:include filename="$(find franka_description)/robots/hand.xacro"/>
+  <xacro:include filename="$(find franka_description)/robots/common/franka_arm.xacro"/>
+  <xacro:include filename="$(find franka_description)/robots/common/franka_hand.xacro"/>
+  <xacro:arg name="arm_id" default="panda" />
   <link name="base_link" />
-  <xacro:panda_arm connected_to="base_link" />
-  <xacro:hand ns="panda" rpy="0 0 ${-pi/4}" connected_to="panda_link8"/>
+  <xacro:franka_arm arm_id="$(arg arm_id)" connected_to="base_link"
+                    joint_limits="${xacro.load_yaml('$(find franka_description)/robots/panda/joint_limits.yaml')}"/>
+  <xacro:franka_hand arm_id="$(arg arm_id)" connected_to="panda_link8"
+                     rpy="0 0 ${-pi/4}" />
 </robot>

File: manipulability_metrics_examples/urdf/timda_dual_arm.xacro (robot description, xacro)
@@ -1,3 +1,32 @@
 <?xml version="1.0" encoding="utf-8"?>
+<robot name="mobile_dual_arm" xmlns:xacro="http://www.ros.org/wiki/xacro">
+  <xacro:include filename="$(find timda_body)/urdf/timda_body.xacro" />
+  <xacro:include filename="$(find single_arm_description)/urdf/single_arm.xacro" />
+  <xacro:include filename="$(find suction_urdf)/urdf/suction_urdf.xacro" />
+  <link name="world"/>
+  <!-- TIMDA body -->
+  <joint name="fixed1" type="fixed">
+    <origin
+      xyz="0 0 0"
+      rpy="0 0 0" />
+    <parent link="world"/>
+    <child link="base_link"/>
+  </joint>
+  <!-- TIMDA right arm with suction tool -->
+  <xacro:single_arm side="r"  parent="slide_right" child="r_tool_link" toolrot="-1.57">
+    <origin xyz="0.0 0.1151 0.0" rpy="1.57 3.1415926 3.1415926" />
+  </xacro:single_arm>
+  <xacro:suction side="r"  parent="r_Link_6">
+    <origin xyz="0 -0.016 0" rpy="0 0 -1.57" />
+  </xacro:suction>
+  <!-- TIMDA left arm with suction tool -->
+  <xacro:single_arm side="l"  parent="slide_left" child="l_tool_link" toolrot="1.57">
+    <origin xyz="0.0 0.1151 0.0" rpy="-1.57 0 0" />
+  </xacro:single_arm>
+  <xacro:suction side="l"  parent="l_Link_6">
+    <origin xyz="0 0.016 0" rpy="0 0 1.57" />
+  </xacro:suction>
+</robot>
+<!-- <?xml version="1.0" encoding="utf-8"?>
 <robot name="mobile_dual_arm" xmlns:xacro="http://www.ros.org/wiki/xacro">
   <xacro:include filename="$(find single_arm_description)/urdf/single_arm.xacro" />
@@ -25,2 +54,3 @@
   </xacro:suction>
 </robot>
+ -->
