Commit message: [ok] timda_dual8, dual manip ellipsoid

File: manipulability_metrics_examples/urdf/timda_dual8.xacro (robot description, xacro)
@@ -14,17 +14,33 @@
   </joint>
   <!-- TIMDA right arm with suction tool -->
-  <xacro:single_arm side="r"  parent="slide_right" child="r_tool_link" toolrot="-1.57">
+  <xacro:single_arm side="r_"  parent="slide_right" child="r_tool_link" toolrot="-1.57">
+    <origin xyz="0.0 0.1151 0.0" rpy="1.57 3.1415926 3.1415926" />
+  </xacro:single_arm>
+  <xacro:suction side="r"  parent="r_tool_link">
+    <origin xyz="0 -0.016 0" rpy="0 0 -1.57" />
+  </xacro:suction>
+  <!-- TIMDA left arm with suction tool -->
+  <xacro:single_arm side="l_"  parent="slide_left" child="l_tool_link" toolrot="1.57">
+    <origin xyz="0.0 0.1151 0.0" rpy="-1.57 0 0" />
+  </xacro:single_arm>
+  <xacro:suction side="l"  parent="l_tool_link">
+    <origin xyz="0 0.016 0" rpy="0 0 1.57" />
+  </xacro:suction>
+  <!-- ======OLD xacro===== -->
+  <!-- TIMDA right arm with suction tool -->
+  <!-- <xacro:single_arm side="r"  parent="slide_right" child="r_tool_link" toolrot="-1.57">
     <origin xyz="0.0 0.1151 0.0" rpy="1.57 3.1415926 3.1415926" />
   </xacro:single_arm>
   <xacro:suction side="r"  >
     <origin xyz="0 -0.016 0" rpy="0 0 -1.57" />
-  </xacro:suction>
+  </xacro:suction> -->
   <!-- TIMDA left arm with suction tool -->
-  <xacro:single_arm side="l"  parent="slide_left" child="l_tool_link" toolrot="1.57">
+  <!-- <xacro:single_arm side="l"  parent="slide_left" child="l_tool_link" toolrot="1.57">
     <origin xyz="0.0 0.1151 0.0" rpy="-1.57 0 0" />
   </xacro:single_arm>
   <xacro:suction side="l"  >
     <origin xyz="0 0.016 0" rpy="0 0 1.57" />
-  </xacro:suction>
+  </xacro:suction> -->
+  <!-- ======OLD xacro===== -->
 </robot>
 <!-- <?xml version="1.0" encoding="utf-8"?>
