Commit message: [ok] organize robot_models

File: robot_models/timda_model/suction_urdf/urdf/suction_urdf.xacro (robot description, xacro)
@@ -3,5 +3,5 @@
   <xacro:include filename="$(find suction_urdf)/urdf/suction.transmission.xacro" />
   <xacro:include filename="$(find suction_urdf)/urdf/suction.gazebo.xacro" />
-  <xacro:macro name="suction" params="side parent *origin">
+  <xacro:macro name="suction" params="side *origin">
     <link
       name="${side}_tool_link">
