Commit message: [tmp] add _d405 gazebo

File: camera_models/realsense2_description/urdf/_d405.gazebo.xacro (robot description, xacro)
@@ -6,11 +6,10 @@
 -->
 <robot xmlns:xacro="http://ros.org/wiki/xacro">
-  <!-- <xacro:macro name="sensor_d405_gazebo" params="name:=camera "> -->
   <xacro:macro name="gazebo_d405" params=" camera_name:=camera
                                            topics_ns:=camera
                                            reference_link
                                            depth_optical_frame
-                                           depth_width:=
-                                           depth_height:=
+                                           depth_width:=1280
+                                           depth_height:=780
                                            depth_fps:=60
                                            color_optical_frame
@@ -18,4 +17,5 @@
                                            color_height:=800
                                            color_fps:=60
+                                           visualize_color:=false
                                            infrared1_optical_frame
                                            infrared2_optical_frame
@@ -23,13 +23,7 @@
                                            infra_height:=720
                                            infra_fps:= 60
-                                           accel_optical_frame
-                                           gyro_optical_frame
-                                           accel_fps:=
-                                           gyro_fps:=
                                            enable_pointCloud:=false
-                                           unite_imu_method:=false
-                                           clip_distance:=
+                                           clip_distance:=0.1
                                            align_depth:=false
-                                           visualize:=false
                                            ">
     <!-- The following values are approximate, and the camera node
@@ -49,16 +43,21 @@
     <xacro:property name="d405_cam_depth_py" value="0"/>
     <xacro:property name="d405_cam_depth_pz" value="${d405_cam_height/2}"/>
-    <!-- **********************************************************-->
-    <!-- GAZEBO DEFINITIONS ***************************************-->
-    <xacro:property name="ir_fps" value="60"/>
+    <!-- ***************************-->
+    <!-- ****GAZEBO DEFINITIONS ****-->
+    <!-- ***************************-->
     <xacro:property name="color_fps" value="60"/>
+    <xacro:property name="infra_fps" value="60"/>
+    <xacro:property name="depth_fps" value="60"/>
     <!-- See realsense datasheet-->
-    <xacro:property name="ir_fov" value="${radians(84)}"/>
     <xacro:property name="color_fov" value="${radians(84)}"/>
+    <xacro:property name="infra_fov" value="${radians(84)}"/>
+    <xacro:property name="depth_fov" value="${radians(84)}"/>
     <!-- Camera image properties -->
-    <xacro:property name="ir_h" value="720"/>
-    <xacro:property name="ir_w" value="1280"/>
-    <xacro:property name="color_h" value="800"/>
-    <xacro:property name="color_w" value="1280"/>
+    <xacro:property name="color_height" value="800"/>
+    <xacro:property name="color_width" value="1280"/>
+    <xacro:property name="infra_height" value="720"/>
+    <xacro:property name="infra_width" value="1280"/>
+    <xacro:property name="depth_height" value="720"/>
+    <xacro:property name="depth_width" value="1280"/>
     <!-- clip_distance -->
     <xacro:property name="min_z" value="0.1"/>
@@ -74,4 +73,5 @@
       <kp>1e+13</kp>
       <kd>1</kd>
+      <!-- Color -->
       <sensor name="${camera_name}color" type="camera">
         <pose frame="">0 ${d405_cam_depth_to_color_offset} 0.0 0 0 0</pose>
@@ -79,6 +79,6 @@
           <horizontal_fov>${color_fov}</horizontal_fov>
           <image>
-            <width>${color_w}</width>
-            <height>${color_h}</height>
+            <width>${color_width}</width>
+            <height>${color_height}</height>
             <format>RGB_INT8</format>
           </image>
@@ -95,13 +95,14 @@
         <always_on>1</always_on>
         <update_rate>${color_fps}</update_rate>
-        <visualize>0</visualize>
-      </sensor>
+        <visualize>${visualize_color}</visualize>
+      </sensor>
+      <!-- InfarRed1:Left -->
       <sensor name="${camera_name}ired1" type="camera">
         <pose frame="">0 ${d405_cam_depth_to_infra1_offset} 0 0 0 0</pose>
         <camera name="${camera_name}">
-          <horizontal_fov>${ir_fov}</horizontal_fov>
-          <image>
-            <width>${ir_w}</width>
-            <height>${ir_h}</height>
+          <horizontal_fov>${infra_fov}</horizontal_fov>
+          <image>
+            <width>${infra_width}</width>
+            <height>${infra_height}</height>
             <format>L_INT8</format>
           </image>
@@ -117,14 +118,15 @@
         </camera>
         <always_on>1</always_on>
-        <update_rate>${ir_fps}</update_rate>
-        <visualize>0</visualize>
-      </sensor>
+        <update_rate>${infra_fps}</update_rate>
+        <visualize>false</visualize>
+      </sensor>
+      <!-- InfarRed2:Right -->
       <sensor name="${camera_name}ired2" type="camera">
         <pose frame="">0 ${d405_cam_depth_to_infra2_offset} 0 0 0 0</pose>
         <camera name="${camera_name}">
-          <horizontal_fov>${ir_fov}</horizontal_fov>
-          <image>
-            <width>${ir_w}</width>
-            <height>${ir_h}</height>
+          <horizontal_fov>${infra_fov}</horizontal_fov>
+          <image>
+            <width>${infra_width}</width>
+            <height>${infra_height}</height>
             <format>L_INT8</format>
           </image>
@@ -140,14 +142,15 @@
         </camera>
         <always_on>1</always_on>
-        <update_rate>${ir_fps}</update_rate>
-        <visualize>0</visualize>
-      </sensor>
+        <update_rate>${infra_fps}</update_rate>
+        <visualize>false</visualize>
+      </sensor>
+      <!-- Depth -->
       <sensor name="${camera_name}depth" type="depth">
         <pose frame="">0 0 0 0 0 0</pose>
         <camera name="${camera_name}">
-          <horizontal_fov>${ir_fov}</horizontal_fov>
-          <image>
-            <width>${ir_w}</width>
-            <height>${ir_h}</height>
+          <horizontal_fov>${depth_fov}</horizontal_fov>
+          <image>
+            <width>${depth_width}</width>
+            <height>${depth_height}</height>
           </image>
           <clip>
@@ -163,11 +166,16 @@
         </camera>
         <always_on>1</always_on>
-        <update_rate>${ir_fps}</update_rate>
-        <visualize>0</visualize>
+        <xacro:unless value="${align_depth}">
+          <update_rate>${depth_fps}</update_rate>
+        </xacro:unless>
+        <xacro:if value="${align_depth}">
+          <update_rate>${color_fps}</update_rate>
+        </xacro:if>
+        <visualize>false</visualize>
       </sensor>
     </gazebo>
     <!-- Load plugin to the model ("robot" in urdf format)-->
     <gazebo>
-      <plugin name="${topic_ns}" filename="librealsense_gazebo_plugin.so">
+      <plugin name="${topics_ns}" filename="librealsense_gazebo_plugin.so">
         <prefix>${camera_name}</prefix>
         <!-- Color camera settings -->
@@ -177,5 +185,5 @@
         <colorCameraInfoTopicName>color/camera_info</colorCameraInfoTopicName>
         <!-- Infrared camera settings -->
-        <infraredUpdateRate>${ir_fps}</infraredUpdateRate>
+        <infraredUpdateRate>${infra_fps}</infraredUpdateRate>
         <infrared1TopicName>infra1/image_raw</infrared1TopicName>
         <infrared2TopicName>infra2/image_raw</infrared2TopicName>
@@ -204,5 +212,5 @@
         <depthOpticalframeName>${camera_name}_depth_optical_frame</depthOpticalframeName> -->
         <!-- Pointlcloud settings -->
-        <pointCloud>false</pointCloud>
+        <pointCloud>${enable_pointCloud}</pointCloud>
         <pointCloudTopicName>depth_registered/points</pointCloudTopicName>
         <!-- <pointCloudTopicName>depth/color/points</pointCloudTopicName> -->

File: camera_models/realsense2_description/urdf/_d405.urdf_prev.xacro (robot description, xacro)
@@ -21,25 +21,7 @@
 <robot name="sensor_d405" xmlns:xacro="http://ros.org/wiki/xacro">
   <!-- Includes -->
-  <xacro:include filename="$(find realsense2_description)/urdf/_d405.gazebo.xacro"/>
   <xacro:include filename="$(find realsense2_description)/urdf/_materials.urdf.xacro" />
   <xacro:include filename="$(find realsense2_description)/urdf/_usb_plug.urdf.xacro" />
-  <xacro:macro name="sensor_d405" params="parent
-                                          use_nominal_extrinsics:=false
-                                          name:=camera
-                                          topics_ns:=camera
-                                          color_width:=1920
-                                          color_height:=1080
-                                          color_fps:=30
-                                          visualize_color:=false
-                                          infra_width:=640
-                                          infra_height:=480
-                                          infra_fps:=30
-                                          clip_distance:=-1.0
-                                          depth_width:=1280
-                                          depth_height:=720
-                                          depth_fps:=30
-                                          align_depth:=false
-                                          enable_pointCloud:=false
-                                          *origin">
+  <xacro:macro name="sensor_d405" params="parent *origin name:=camera use_nominal_extrinsics:=false">
     <xacro:arg name="add_plug" default="false" />
     <xacro:property name="M_PI" value="3.1415926535897931" />
@@ -156,5 +138,4 @@
       <link name="${name}_color_optical_frame"/>
     </xacro:if>
-    <!-- usb_plug -->
     <xacro:if value="$(arg add_plug)">
       <xacro:usb_plug parent="${name}_link" name="${name}_usb_plug">
@@ -162,26 +143,4 @@
       </xacro:usb_plug>
     </xacro:if>
-    <!-- Realsense Gazebo Plugin -->
-    <xacro:gazebo_d405 camera_name="${name}"
-                        topics_ns="${topics_ns}"
-                        reference_link="${name}_link"
-                        depth_optical_frame="${name}_depth_optical_frame"
-                        depth_width="${depth_width}"
-                        depth_height="${depth_height}"
-                        depth_fps="${depth_fps}"
-                        color_optical_frame="${name}_color_optical_frame"
-                        color_width="${color_width}"
-                        color_height="${color_height}"
-                        color_fps="${color_fps}"
-                        visualize_color="${visualize_color}"
-                        infrared1_optical_frame="${name}_left_ir_optical_frame"
-                        infrared2_optical_frame="${name}_right_ir_optical_frame"
-                        infra_width="${infra_width}"
-                        infra_height="${infra_height}"
-                        infra_fps="${infra_fps}"
-                        enable_pointCloud="${enable_pointCloud}"
-                        clip_distance="${clip_distance}"
-                        align_depth="${align_depth}"
-    />
   </xacro:macro>
 </robot>

File: camera_models/realsense2_description/urdf/_d435i.urdf.xacro (robot description, xacro)
@@ -1,30 +1,194 @@
 <?xml version="1.0"?>
 <!--
-# Copyright 2023 Intel Corporation. All Rights Reserved.
-#
-# Licensed under the Apache License, Version 2.0 (the "License");
-# you may not use this file except in compliance with the License.
-# You may obtain a copy of the License at
-#
-#     http://www.apache.org/licenses/LICENSE-2.0
-#
-# Unless required by applicable law or agreed to in writing, software
-# distributed under the License is distributed on an "AS IS" BASIS,
-# WITHOUT WARRANTIES OR CONDITIONS OF ANY KIND, either express or implied.
-# See the License for the specific language governing permissions and
-# limitations under the License.
--->
-<!--
-This is the URDF model for the Intel RealSense 435i camera, in it's
+Aknolegment: This file was copied from the realsense repository of
+pal-robotics-forks( https://github.com/pal-robotics-forks/realsense/ ).
+and then modified.
+License: Apache 2.0. See LICENSE file in root directory.
+Copyright(c) 2017 Intel Corporation. All Rights Reserved
+This is the URDF model for the Intel RealSense 430 camera, in it's
 aluminum peripherial evaluation case.
 -->
 <robot name="sensor_d435i" xmlns:xacro="http://ros.org/wiki/xacro">
-  <xacro:include filename="$(find realsense2_description)/urdf/_d435.urdf.xacro"/>
-  <xacro:include filename="$(find realsense2_description)/urdf/_d435i_imu_modules.urdf.xacro"/>
-  <xacro:macro name="sensor_d435i" params="parent *origin name:=camera use_nominal_extrinsics:=false">
-    <xacro:sensor_d435 parent="${parent}" name="${name}" use_nominal_extrinsics="${use_nominal_extrinsics}">
-      <xacro:insert_block name="origin" />
-    </xacro:sensor_d435>
-    <xacro:d435i_imu_modules name="${name}" use_nominal_extrinsics="${use_nominal_extrinsics}"/>
+  <!--File includes-->
+  <xacro:include filename="$(find realsense_gazebo_description)/urdf/_d435i.gazebo.xacro"/>
+  <xacro:macro name="sensor_d435i" params="parent
+                                          name:=camera
+                                          topics_ns:=camera
+                                          color_width:=1920
+                                          color_height:=1080
+                                          color_fps:=30
+                                          visualize_color:=false
+                                          infra_width:=640
+                                          infra_height:=480
+                                          infra_fps:=30
+                                          clip_distance:=-1.0
+                                          depth_width:=1280
+                                          depth_height:=720
+                                          depth_fps:=30
+                                          unite_imu_method:=false
+                                          accel_fps:=250
+                                          gyro_fps:=400
+                                          align_depth:=false
+                                          enable_pointCloud:=false
+                                          *origin">
+    <xacro:property name="M_PI" value="3.1415926535897931"/>
+    <!-- The following values are approximate, and the camera node
+     publishing TF values with actual calibrated camera extrinsic values -->
+    <xacro:property name="d435i_cam_depth_to_left_ir_offset" value="0.0"/>
+    <xacro:property name="d435i_cam_depth_to_right_ir_offset" value="-0.050"/>
+    <xacro:property name="d435i_cam_depth_to_color_offset" value="0.015"/>
+    <!-- The following values model the aluminum peripherial case for the
+  	D435 camera, with the camera joint represented by the actual
+  	peripherial camera tripod mount -->
+    <xacro:property name="d435i_cam_width" value="0.090"/>
+    <xacro:property name="d435i_cam_height" value="0.025"/>
+    <xacro:property name="d435i_cam_depth" value="0.02505"/>
+    <xacro:property name="d435i_cam_mount_from_center_offset" value="0.0149"/>
+    <!-- The following offset is relative the the physical D435 camera peripherial
+  	camera tripod mount -->
+    <xacro:property name="d435i_cam_depth_px" value="${d435i_cam_mount_from_center_offset}"/>
+    <xacro:property name="d435i_cam_depth_py" value="0.0175"/>
+    <xacro:property name="d435i_cam_depth_pz" value="${d435i_cam_height/2}"/>
+    <material name="${name}_aluminum">
+	  <color rgba="0.5 0.5 0.5 1"/>
+    </material>
+    <!-- camera body, with origin at bottom screw mount -->
+    <joint name="${name}_joint" type="fixed">
+      <xacro:insert_block name="origin"/>
+      <parent link="${parent}"/>
+      <child link="${name}_bottom_screw_frame"/>
+    </joint>
+    <link name="${name}_bottom_screw_frame"/>
+    <joint name="${name}_link_joint" type="fixed">
+      <origin xyz="0 ${d435i_cam_depth_py} ${d435i_cam_depth_pz}" rpy="0 0 0"/>
+      <parent link="${name}_bottom_screw_frame"/>
+      <child link="${name}_link"/>
+    </joint>
+    <link name="${name}_link">
+      <visual>
+      <origin xyz="${d435i_cam_mount_from_center_offset} ${-d435i_cam_depth_py} 0" rpy="${M_PI/2} 0 ${M_PI/2}"/>
+        <geometry>
+          <mesh filename="package://realsense_gazebo_description/meshes/d435.dae"/>
+        </geometry>
+        <material name="${name}_aluminum"/>
+      </visual>
+      <collision>
+        <origin xyz="0 ${-d435i_cam_depth_py} 0" rpy="0 0 0"/>
+        <geometry>
+        <box size="${d435i_cam_depth} ${d435i_cam_width} ${d435i_cam_height}"/>
+        </geometry>
+      </collision>
+      <inertial>
+        <!-- The following are not reliable values, and should not be used for modeling -->
+        <mass value="0.564"/>
+        <origin xyz="0 0 0"/>
+        <inertia ixx="0.003881243" ixy="0.0" ixz="0.0" iyy="0.000498940" iyz="0.0" izz="0.003879257"/>
+      </inertial>
+    </link>
+    <!-- camera depth joints and links -->
+    <joint name="${name}_depth_joint" type="fixed">
+      <origin xyz="0 0 0" rpy="0 0 0"/>
+      <parent link="${name}_link"/>
+      <child link="${name}_depth_frame"/>
+    </joint>
+    <link name="${name}_depth_frame"/>
+    <joint name="${name}_depth_optical_joint" type="fixed">
+      <origin xyz="0 0 0" rpy="${-M_PI/2} 0 ${-M_PI/2}"/>
+      <parent link="${name}_depth_frame"/>
+      <child link="${name}_depth_optical_frame"/>
+    </joint>
+    <link name="${name}_depth_optical_frame"/>
+    <!-- camera left IR joints and links -->
+    <joint name="${name}_left_ir_joint" type="fixed">
+      <origin xyz="0 ${d435i_cam_depth_to_left_ir_offset} 0" rpy="0 0 0"/>
+      <parent link="${name}_depth_frame"/>
+      <child link="${name}_left_ir_frame"/>
+    </joint>
+    <link name="${name}_left_ir_frame"/>
+    <joint name="${name}_left_ir_optical_joint" type="fixed">
+      <origin xyz="0 0 0" rpy="${-M_PI/2} 0 ${-M_PI/2}"/>
+      <parent link="${name}_left_ir_frame"/>
+      <child link="${name}_left_ir_optical_frame"/>
+    </joint>
+    <link name="${name}_left_ir_optical_frame"/>
+    <!-- camera right IR joints and links -->
+    <joint name="${name}_right_ir_joint" type="fixed">
+      <origin xyz="0 ${d435i_cam_depth_to_right_ir_offset} 0" rpy="0 0 0"/>
+      <parent link="${name}_depth_frame"/>
+      <child link="${name}_right_ir_frame"/>
+    </joint>
+    <link name="${name}_right_ir_frame"/>
+    <joint name="${name}_right_ir_optical_joint" type="fixed">
+      <origin xyz="0 0 0" rpy="${-M_PI/2} 0 ${-M_PI/2}"/>
+      <parent link="${name}_right_ir_frame"/>
+      <child link="${name}_right_ir_optical_frame"/>
+    </joint>
+    <link name="${name}_right_ir_optical_frame"/>
+    <!-- camera color joints and links -->
+    <joint name="${name}_color_joint" type="fixed">
+      <origin xyz="0 ${d435i_cam_depth_to_color_offset} 0" rpy="0 0 0"/>
+      <parent link="${name}_depth_frame"/>
+      <child link="${name}_color_frame"/>
+    </joint>
+    <link name="${name}_color_frame"/>
+    <joint name="${name}_color_optical_joint" type="fixed">
+      <origin xyz="0 0 0" rpy="${-M_PI/2} 0 ${-M_PI/2}"/>
+      <parent link="${name}_color_frame"/>
+      <child link="${name}_color_optical_frame"/>
+    </joint>
+    <link name="${name}_color_optical_frame"/>
+    <!-- camera accel joints and links -->
+    <joint name="${name}_accel_joint" type="fixed">
+      <origin xyz="-0.00174 0.00552 0.0176" rpy="0 0 0"/>
+      <parent link="${name}_link"/>
+      <child link="${name}_accel_frame"/>
+    </joint>
+    <link name="${name}_accel_frame"/>
+    <joint name="${name}_accel_optical_joint" type="fixed">
+      <origin xyz="0 0 0" rpy="${-M_PI/2} 0 ${-M_PI/2}"/>
+      <parent link="${name}_accel_frame"/>
+      <child link="${name}_accel_optical_frame"/>
+    </joint>
+    <link name="${name}_accel_optical_frame"/>
+    <!-- camera gyro joints and links -->
+    <joint name="${name}_gyro_joint" type="fixed">
+      <origin xyz="-0.00174 0.00552 0.0176" rpy="0 0 0"/>
+      <parent link="${name}_link"/>
+      <child link="${name}_gyro_frame"/>
+    </joint>
+    <link name="${name}_gyro_frame"/>
+    <joint name="${name}_gyro_optical_joint" type="fixed">
+      <origin xyz="0 0 0" rpy="${-M_PI/2} 0 ${-M_PI/2}"/>
+      <parent link="${name}_gyro_frame"/>
+      <child link="${name}_gyro_optical_frame"/>
+    </joint>
+    <link name="${name}_gyro_optical_frame"/>
+    <!-- Realsense Gazebo Plugin -->
+    <xacro:gazebo_d435i camera_name="${name}"
+                        topics_ns="${topics_ns}"
+                        reference_link="${name}_link"
+                        depth_optical_frame="${name}_depth_optical_frame"
+                        depth_width="${depth_width}"
+                        depth_height="${depth_height}"
+                        depth_fps="${depth_fps}"
+                        color_optical_frame="${name}_color_optical_frame"
+                        color_width="${color_width}"
+                        color_height="${color_height}"
+                        color_fps="${color_fps}"
+                        visualize_color="${visualize_color}"
+                        infrared1_optical_frame="${name}_left_ir_optical_frame"
+                        infrared2_optical_frame="${name}_right_ir_optical_frame"
+                        infra_width="${infra_width}"
+                        infra_height="${infra_height}"
+                        infra_fps="${infra_fps}"
+                        accel_optical_frame="${name}_accel_optical_frame"
+                        gyro_optical_frame="${name}_gyro_optical_frame"
+                        accel_fps="${accel_fps}"
+                        gyro_fps="${gyro_fps}"
+                        enable_pointCloud="${enable_pointCloud}"
+                        unite_imu_method="${unite_imu_method}"
+                        clip_distance="${clip_distance}"
+                        align_depth="${align_depth}"
+    />
   </xacro:macro>
 </robot>
