Commit message: [ok] d405, d435i rgb, color pointcloud ok

File: camera_models/realsense2_description/urdf/_d405.gazebo.xacro (robot description, xacro)
@@ -24,5 +24,6 @@
                                            infra_fps:= 60
                                            enable_pointCloud:=false
-                                           clip_distance:=0.1
+                                           clip_distance_z_min:=0.1
+                                           clip_distance_z_max:=-0.1
                                            align_depth:=false
                                            ">
@@ -60,7 +61,7 @@
     <xacro:property name="depth_height" value="720"/>
     <xacro:property name="depth_width" value="1280"/>
-    <!-- clip_distance -->
-    <xacro:property name="min_z" value="0.1"/>
-    <xacro:property name="max_z" value="0.5"/>
+    <!-- clip_distance_z -->
+    <!-- <xacro:property name="clip_distance_z_min" value="0.1"/>
+    <xacro:property name="clip_distance_z_max" value="0.5"/> -->
     <!-- Load parameters to model's main link-->
     <gazebo reference="${camera_name}_link">
@@ -149,12 +150,27 @@
         <pose frame="">0 0 0 0 0 0</pose>
         <camera name="${camera_name}">
-          <horizontal_fov>${depth_fov}</horizontal_fov>
-          <image>
-            <width>${depth_width}</width>
-            <height>${depth_height}</height>
-          </image>
-          <clip>
-            <near>${min_z}</near>
-            <far>${max_z}</far>
+          <!-- align-depth settings -->
+          <xacro:unless value="${align_depth}">
+            <horizontal_fov>${depth_fov}</horizontal_fov>
+            <image>
+              <width>${depth_width}</width>
+              <height>${depth_height}</height>
+            </image>
+          </xacro:unless>
+          <xacro:if value="${align_depth}">
+            <horizontal_fov>${color_fov}</horizontal_fov>
+            <image>
+              <width>${color_width}</width>
+              <height>${color_height}</height>
+            </image>
+          </xacro:if>
+          <clip>
+            <near>${clip_distance_z_min}</near>
+            <xacro:unless value="${clip_distance_z_max > 0.0}">
+              <far>100</far>
+            </xacro:unless>
+            <xacro:if value="${clip_distance_z_max > 0.0}">
+              <far>${clip_distance_z_max}</far>
+            </xacro:if>
           </clip>
           <noise>
@@ -195,5 +211,10 @@
         <depthUpdateRate>${depth_fps}</depthUpdateRate>
         <rangeMinDepth>0.2</rangeMinDepth>
-        <rangeMaxDepth>10.0</rangeMaxDepth>
+        <xacro:unless value="${clip_distance_z_max > 0.0}">
+          <rangeMaxDepth>10.0</rangeMaxDepth>
+        </xacro:unless>
+        <xacro:if value="${clip_distance_z_max > 0.0}">
+          <rangeMaxDepth>${clip_distance_z_max}</rangeMaxDepth>
+        </xacro:if>
         <xacro:unless value="${align_depth}">
         	<depthUpdateRate>${depth_fps}</depthUpdateRate>
@@ -216,5 +237,5 @@
         <!-- <pointCloudTopicName>depth/color/points</pointCloudTopicName> -->
         <!-- <pointCloudTopicName>/camera/depth_registered/points</pointCloudTopicName> -->
-        <pointCloudCutoff>0.5</pointCloudCutoff>
+        <pointCloudCutoff>0.1</pointCloudCutoff>
       </plugin>
     </gazebo>

File: camera_models/realsense2_description/urdf/_d405.urdf.xacro (robot description, xacro)
@@ -35,5 +35,6 @@
                                           infra_height:=480
                                           infra_fps:=30
-                                          clip_distance:=-1.0
+                                          clip_distance_z_min:=0.1
+                                          clip_distance_z_max:=-1.0
                                           depth_width:=1280
                                           depth_height:=720
@@ -42,5 +43,5 @@
                                           enable_pointCloud:=false
                                           *origin">
-    <xacro:arg name="add_plug" default="false" />
+    <!-- <xacro:arg name="add_plug" default="false" /> -->
     <xacro:property name="M_PI" value="3.1415926535897931" />
     <!-- The following values are approximate, and the camera node
@@ -157,9 +158,9 @@
     </xacro:if>
     <!-- usb_plug -->
-    <xacro:if value="$(arg add_plug)">
+    <!-- <xacro:if value="$(arg add_plug)">
       <xacro:usb_plug parent="${name}_link" name="${name}_usb_plug">
         <origin xyz="${-0.00153-d405_mesh_x_offset} ${d405_cam_width/2-d405_cam_depth_py} 0" rpy="${M_PI} 0 0"/>
       </xacro:usb_plug>
-    </xacro:if>
+    </xacro:if> -->
     <!-- Realsense Gazebo Plugin -->
     <xacro:gazebo_d405 camera_name="${name}"
@@ -181,5 +182,6 @@
                         infra_fps="${infra_fps}"
                         enable_pointCloud="${enable_pointCloud}"
-                        clip_distance="${clip_distance}"
+                        clip_distance_z_min="${clip_distance_z_min}"
+                        clip_distance_z_max="${clip_distance_z_max}"
                         align_depth="${align_depth}"
     />

File: camera_models/realsense2_description/urdf/_d435.gazebo.xacro (robot description, xacro)
@@ -6,34 +6,29 @@
 License: Apache 2.0. See LICENSE file in root directory.
 Copyright(c) 2017 PAL Robotics, S.L. All Rights Reserved
-This is the Gazebo URDF model for the Intel RealSense D435i camera
+This is the Gazebo URDF model for the Intel RealSense D435 camera
 -->
 <robot xmlns:xacro="http://ros.org/wiki/xacro">
-  <xacro:macro name="gazebo_d435i" params=" camera_name:=camera
-                                            topics_ns:=camera
-                                            reference_link
-                                            depth_optical_frame
-                                            depth_width:=1280
-                                            depth_height:=720
-                                            depth_fps:=30
-                                            color_optical_frame
-                                            color_width:=1920
-                                            color_height:=1080
-                                            color_fps:=30
-                                            visualize_color:=false
-                                            infrared1_optical_frame
-                                            infrared2_optical_frame
-                                            infra_width:=640
-                                            infra_height:=480
-                                            infra_fps:=30
-                                            accel_optical_frame
-                                            gyro_optical_frame
-                                            accel_fps:=250
-                                            gyro_fps:=400
-                                            enable_pointCloud:=false
-                                            unite_imu_method:=false
-                                            clip_distance_z_min:=0.1
-                                            clip_distance_z_max:=-1.0
-                                            align_depth:=false
-                                            ">
+  <xacro:macro name="gazebo_d435" params="reference_link
+                                          camera_name:=camera
+                                          topics_ns:=camera
+                                          depth_optical_frame
+                                          color_optical_frame
+                                          infrared1_optical_frame
+                                          infrared2_optical_frame
+                                          clip_distance_z_min:=0.1
+                                          clip_distance_z_max:=-1.0
+                                          depth_width:=1280
+                                          depth_height:=720
+                                          depth_fps:=30
+                                          color_width:=1920
+                                          color_height:=1080
+                                          color_fps:=30
+                                          infra_width:=640
+                                          infra_height:=480
+                                          infra_fps:=30
+                                          align_depth:=false
+                                          enable_pointCloud:=false
+                                          visualize:=false
+                                          ">
     <!-- Load parameters to model's main link-->
     <xacro:property name="deg_to_rad" value="0.01745329251994329577"/>
@@ -52,5 +47,4 @@
       <!--<max_vel>0.01</max_vel>
       <min_depth>0</min_depth>-->
-      <!-- Color -->
       <sensor name="${camera_name}color" type="camera">
         <camera name="${camera_name}">
@@ -73,7 +67,6 @@
         <always_on>1</always_on>
         <update_rate>${color_fps}</update_rate>
-        <visualize>${visualize_color}</visualize>
-      </sensor>
-      <!-- InfarRed1 -->
+        <visualize>${visualize}</visualize>
+      </sensor>
       <sensor name="${camera_name}ired1" type="camera">
         <camera name="${camera_name}">
@@ -98,5 +91,4 @@
         <visualize>false</visualize>
       </sensor>
-      <!-- InfarRed2 -->
       <sensor name="${camera_name}ired2" type="camera">
         <camera name="${camera_name}">
@@ -121,5 +113,4 @@
         <visualize>false</visualize>
       </sensor>
-      <!-- Depth -->
       <sensor name="${camera_name}depth" type="depth">
         <camera name="${camera_name}">
@@ -141,9 +132,9 @@
           <clip>
             <near>0.1</near>
-            <xacro:unless value="${clip_distance_z_max > 0.0}">
+            <xacro:unless value="${clip_distance_z_m > 0.0}">
               <far>100</far>
             </xacro:unless>
-            <xacro:if value="${clip_distance_z_max > 0.0}">
-              <far>${clip_distance_z_max}</far>
+            <xacro:if value="${clip_distance_z_m > 0.0}">
+              <far>${clip_distance_z_m}</far>
             </xacro:if>
           </clip>
@@ -163,57 +154,5 @@
         <visualize>false</visualize>
       </sensor>
-      <!-- IMU -->
-      <xacro:if value="${unite_imu_method == 'copy' or unite_imu_method == 'linear_interpolation'}">
-        <sensor name="${camera_name}imu" type="imu">
-          <always_on>true</always_on>
-          <update_rate>${gyro_fps}</update_rate>
-          <topic>${camera_name}/imu/sample</topic>
-          <plugin name="{camera_name}imu" filename="libgazebo_ros_imu_sensor.so">
-            <topicName>${camera_name}/imu/sample</topicName>
-            <bodyName>${camera_name}_link</bodyName>
-            <frameName>${gyro_optical_frame}</frameName>
-            <updateRateHZ>${gyro_fps}</updateRateHZ>
-            <gaussianNoise>0.1</gaussianNoise>
-            <xyzOffset>0 0 0</xyzOffset>
-            <rpyOffset>0 0 0</rpyOffset>
-          </plugin>
-        </sensor>
-      </xacro:if>
-      <!-- Accel and gyro -->
-      <xacro:unless value="${unite_imu_method == 'copy' or unite_imu_method == 'linear_interpolation'}">
-        <sensor name="{camera_name}accel" type="imu">
-          <always_on>true</always_on>
-          <update_rate>${accel_fps}</update_rate>
-          <topic>${camera_name}/accel/sample</topic>
-          <plugin name="${topics_ns}_accel_plugin" filename="librealsense_gazebo_accel_sensor.so">
-            <topicName>${camera_name}/accel/sample</topicName>
-            <bodyName>${camera_name}_link</bodyName>
-            <updateRateHZ>${accel_fps}</updateRateHZ>
-            <gaussianNoise>0.1</gaussianNoise>
-            <xyzOffset>0 0 0</xyzOffset>
-            <rpyOffset>0 0 0</rpyOffset>
-            <frameName>${accel_optical_frame}</frameName>
-            <initialOrientationAsReference>false</initialOrientationAsReference>
-          </plugin>
-          <pose>0 0 0 0 0 0</pose>
-        </sensor>
-        <sensor name="{camera_name}gyro" type="imu">
-          <always_on>true</always_on>
-          <update_rate>${gyro_fps}</update_rate>
-          <topic>${camera_name}/gyro/sample</topic>
-          <plugin name="${topics_ns}_gyro_plugin" filename="librealsense_gazebo_gyro_sensor.so">
-            <topicName>${camera_name}/gyro/sample</topicName>
-            <bodyName>${camera_name}_link</bodyName>
-            <updateRateHZ>${gyro_fps}</updateRateHZ>
-            <gaussianNoise>0.1</gaussianNoise>
-            <xyzOffset>0 0 0</xyzOffset>
-            <rpyOffset>0 0 0</rpyOffset>
-            <frameName>${gyro_optical_frame}</frameName>
-            <initialOrientationAsReference>false</initialOrientationAsReference>
-          </plugin>
-        </sensor>
-      </xacro:unless>
     </gazebo>
-    <!-- Load plugin to the model ("robot" in urdf format)-->
     <gazebo>
       <plugin name="${topics_ns}" filename="librealsense_gazebo_plugin.so">
@@ -234,9 +173,9 @@
         <!-- Depth camera settings -->
       	<rangeMinDepth>0.2</rangeMinDepth>
-        <xacro:unless value="${clip_distance_z_max > 0.0}">
+        <xacro:unless value="${clip_distance_z_m > 0.0}">
       	  <rangeMaxDepth>10.0</rangeMaxDepth>
         </xacro:unless>
-        <xacro:if value="${clip_distance_z_max > 0.0}">
-          <rangeMaxDepth>${clip_distance_z_max}</rangeMaxDepth>
+        <xacro:if value="${clip_distance_z_m > 0.0}">
+          <rangeMaxDepth>${clip_distance_z_m}</rangeMaxDepth>
         </xacro:if>
         <xacro:unless value="${align_depth}">
@@ -254,8 +193,6 @@
         <!-- Pointlcloud settings -->
       	<pointCloud>${enable_pointCloud}</pointCloud>
-        <pointCloudTopicName>depth_registered/points</pointCloudTopicName>
-        <!-- <pointCloudTopicName>depth/color/points</pointCloudTopicName> -->
-        <!-- <pointCloudTopicName>/camera/depth_registered/points</pointCloudTopicName> -->
-        <pointCloudCutoff>0.1</pointCloudCutoff>
+      	<pointCloudTopicName>depth/color/points</pointCloudTopicName>
+      	<pointCloudCutoff>0.5</pointCloudCutoff>
       </plugin>
     </gazebo>

File: camera_models/realsense2_description/urdf/_d435i.urdf.xacro (robot description, xacro)
@@ -13,4 +13,5 @@
   <xacro:include filename="$(find realsense_gazebo_description)/urdf/_d435i.gazebo.xacro"/>
   <xacro:macro name="sensor_d435i" params="parent
+                                          use_nominal_extrinsics:=false
                                           name:=camera
                                           topics_ns:=camera
@@ -22,5 +23,6 @@
                                           infra_height:=480
                                           infra_fps:=30
-                                          clip_distance:=-1.0
+                                          clip_distance_z_min:=0.1
+                                          clip_distance_z_max:=-1.0
                                           depth_width:=1280
                                           depth_height:=720
@@ -86,82 +88,85 @@
       </inertial>
     </link>
-    <!-- camera depth joints and links -->
-    <joint name="${name}_depth_joint" type="fixed">
-      <origin xyz="0 0 0" rpy="0 0 0"/>
-      <parent link="${name}_link"/>
-      <child link="${name}_depth_frame"/>
-    </joint>
-    <link name="${name}_depth_frame"/>
-    <joint name="${name}_depth_optical_joint" type="fixed">
-      <origin xyz="0 0 0" rpy="${-M_PI/2} 0 ${-M_PI/2}"/>
-      <parent link="${name}_depth_frame"/>
-      <child link="${name}_depth_optical_frame"/>
-    </joint>
-    <link name="${name}_depth_optical_frame"/>
-    <!-- camera left IR joints and links -->
-    <joint name="${name}_left_ir_joint" type="fixed">
-      <origin xyz="0 ${d435i_cam_depth_to_left_ir_offset} 0" rpy="0 0 0"/>
-      <parent link="${name}_depth_frame"/>
-      <child link="${name}_left_ir_frame"/>
-    </joint>
-    <link name="${name}_left_ir_frame"/>
-    <joint name="${name}_left_ir_optical_joint" type="fixed">
-      <origin xyz="0 0 0" rpy="${-M_PI/2} 0 ${-M_PI/2}"/>
-      <parent link="${name}_left_ir_frame"/>
-      <child link="${name}_left_ir_optical_frame"/>
-    </joint>
-    <link name="${name}_left_ir_optical_frame"/>
-    <!-- camera right IR joints and links -->
-    <joint name="${name}_right_ir_joint" type="fixed">
-      <origin xyz="0 ${d435i_cam_depth_to_right_ir_offset} 0" rpy="0 0 0"/>
-      <parent link="${name}_depth_frame"/>
-      <child link="${name}_right_ir_frame"/>
-    </joint>
-    <link name="${name}_right_ir_frame"/>
-    <joint name="${name}_right_ir_optical_joint" type="fixed">
-      <origin xyz="0 0 0" rpy="${-M_PI/2} 0 ${-M_PI/2}"/>
-      <parent link="${name}_right_ir_frame"/>
-      <child link="${name}_right_ir_optical_frame"/>
-    </joint>
-    <link name="${name}_right_ir_optical_frame"/>
-    <!-- camera color joints and links -->
-    <joint name="${name}_color_joint" type="fixed">
-      <origin xyz="0 ${d435i_cam_depth_to_color_offset} 0" rpy="0 0 0"/>
-      <parent link="${name}_depth_frame"/>
-      <child link="${name}_color_frame"/>
-    </joint>
-    <link name="${name}_color_frame"/>
-    <joint name="${name}_color_optical_joint" type="fixed">
-      <origin xyz="0 0 0" rpy="${-M_PI/2} 0 ${-M_PI/2}"/>
-      <parent link="${name}_color_frame"/>
-      <child link="${name}_color_optical_frame"/>
-    </joint>
-    <link name="${name}_color_optical_frame"/>
-    <!-- camera accel joints and links -->
-    <joint name="${name}_accel_joint" type="fixed">
-      <origin xyz="-0.00174 0.00552 0.0176" rpy="0 0 0"/>
-      <parent link="${name}_link"/>
-      <child link="${name}_accel_frame"/>
-    </joint>
-    <link name="${name}_accel_frame"/>
-    <joint name="${name}_accel_optical_joint" type="fixed">
-      <origin xyz="0 0 0" rpy="${-M_PI/2} 0 ${-M_PI/2}"/>
-      <parent link="${name}_accel_frame"/>
-      <child link="${name}_accel_optical_frame"/>
-    </joint>
-    <link name="${name}_accel_optical_frame"/>
-    <!-- camera gyro joints and links -->
-    <joint name="${name}_gyro_joint" type="fixed">
-      <origin xyz="-0.00174 0.00552 0.0176" rpy="0 0 0"/>
-      <parent link="${name}_link"/>
-      <child link="${name}_gyro_frame"/>
-    </joint>
-    <link name="${name}_gyro_frame"/>
-    <joint name="${name}_gyro_optical_joint" type="fixed">
-      <origin xyz="0 0 0" rpy="${-M_PI/2} 0 ${-M_PI/2}"/>
-      <parent link="${name}_gyro_frame"/>
-      <child link="${name}_gyro_optical_frame"/>
-    </joint>
-    <link name="${name}_gyro_optical_frame"/>
+    <!-- Use the nominal extrinsics between camera frames if the calibrated extrinsics aren't being published. e.g. running the device in simulation  -->
+    <xacro:if value="${use_nominal_extrinsics}">
+      <!-- camera depth joints and links -->
+      <joint name="${name}_depth_joint" type="fixed">
+        <origin xyz="0 0 0" rpy="0 0 0"/>
+        <parent link="${name}_link"/>
+        <child link="${name}_depth_frame"/>
+      </joint>
+      <link name="${name}_depth_frame"/>
+      <joint name="${name}_depth_optical_joint" type="fixed">
+        <origin xyz="0 0 0" rpy="${-M_PI/2} 0 ${-M_PI/2}"/>
+        <parent link="${name}_depth_frame"/>
+        <child link="${name}_depth_optical_frame"/>
+      </joint>
+      <link name="${name}_depth_optical_frame"/>
+      <!-- camera left IR joints and links -->
+      <joint name="${name}_left_ir_joint" type="fixed">
+        <origin xyz="0 ${d435i_cam_depth_to_left_ir_offset} 0" rpy="0 0 0"/>
+        <parent link="${name}_depth_frame"/>
+        <child link="${name}_left_ir_frame"/>
+      </joint>
+      <link name="${name}_left_ir_frame"/>
+      <joint name="${name}_left_ir_optical_joint" type="fixed">
+        <origin xyz="0 0 0" rpy="${-M_PI/2} 0 ${-M_PI/2}"/>
+        <parent link="${name}_left_ir_frame"/>
+        <child link="${name}_left_ir_optical_frame"/>
+      </joint>
+      <link name="${name}_left_ir_optical_frame"/>
+      <!-- camera right IR joints and links -->
+      <joint name="${name}_right_ir_joint" type="fixed">
+        <origin xyz="0 ${d435i_cam_depth_to_right_ir_offset} 0" rpy="0 0 0"/>
+        <parent link="${name}_depth_frame"/>
+        <child link="${name}_right_ir_frame"/>
+      </joint>
+      <link name="${name}_right_ir_frame"/>
+      <joint name="${name}_right_ir_optical_joint" type="fixed">
+        <origin xyz="0 0 0" rpy="${-M_PI/2} 0 ${-M_PI/2}"/>
+        <parent link="${name}_right_ir_frame"/>
+        <child link="${name}_right_ir_optical_frame"/>
+      </joint>
+      <link name="${name}_right_ir_optical_frame"/>
+      <!-- camera color joints and links -->
+      <joint name="${name}_color_joint" type="fixed">
+        <origin xyz="0 ${d435i_cam_depth_to_color_offset} 0" rpy="0 0 0"/>
+        <parent link="${name}_depth_frame"/>
+        <child link="${name}_color_frame"/>
+      </joint>
+      <link name="${name}_color_frame"/>
+      <joint name="${name}_color_optical_joint" type="fixed">
+        <origin xyz="0 0 0" rpy="${-M_PI/2} 0 ${-M_PI/2}"/>
+        <parent link="${name}_color_frame"/>
+        <child link="${name}_color_optical_frame"/>
+      </joint>
+      <link name="${name}_color_optical_frame"/>
+      <!-- camera accel joints and links -->
+      <joint name="${name}_accel_joint" type="fixed">
+        <origin xyz="-0.00174 0.00552 0.0176" rpy="0 0 0"/>
+        <parent link="${name}_link"/>
+        <child link="${name}_accel_frame"/>
+      </joint>
+      <link name="${name}_accel_frame"/>
+      <joint name="${name}_accel_optical_joint" type="fixed">
+        <origin xyz="0 0 0" rpy="${-M_PI/2} 0 ${-M_PI/2}"/>
+        <parent link="${name}_accel_frame"/>
+        <child link="${name}_accel_optical_frame"/>
+      </joint>
+      <link name="${name}_accel_optical_frame"/>
+      <!-- camera gyro joints and links -->
+      <joint name="${name}_gyro_joint" type="fixed">
+        <origin xyz="-0.00174 0.00552 0.0176" rpy="0 0 0"/>
+        <parent link="${name}_link"/>
+        <child link="${name}_gyro_frame"/>
+      </joint>
+      <link name="${name}_gyro_frame"/>
+      <joint name="${name}_gyro_optical_joint" type="fixed">
+        <origin xyz="0 0 0" rpy="${-M_PI/2} 0 ${-M_PI/2}"/>
+        <parent link="${name}_gyro_frame"/>
+        <child link="${name}_gyro_optical_frame"/>
+      </joint>
+      <link name="${name}_gyro_optical_frame"/>
+    </xacro:if>
     <!-- Realsense Gazebo Plugin -->
     <xacro:gazebo_d435i camera_name="${name}"
@@ -188,5 +193,6 @@
                         enable_pointCloud="${enable_pointCloud}"
                         unite_imu_method="${unite_imu_method}"
-                        clip_distance="${clip_distance}"
+                        clip_distance_z_min="${clip_distance_z_min}"
+                        clip_distance_z_max="${clip_distance_z_max}"
                         align_depth="${align_depth}"
     />
