Commit message: [tmp] cam_ur5e_gripper

File: robot_models/universal_robots/ur_description/urdf/ur5e_cam_gripper.urdf.xacro (robot description, xacro)
@@ -27,6 +27,5 @@
     <origin xyz="0 0 0" rpy="0 -1.5707963268 0"/>
   </xacro:sensor_d405> -->
-  <!-- <xacro:sensor_d405 parent="flange"  -->
-  <xacro:sensor_d405 parent="wrist_3_link"
+  <xacro:sensor_d405 parent="flange"
                      name="$(arg name)"
                      topics_ns="$(arg topics_ns)"
@@ -35,6 +34,13 @@
                      align_depth="$(arg align_depth)"
                      enable_pointCloud="$(arg enable_pointCloud)">
-    <!-- <origin xyz="0 0 0" rpy="0 -1.5707963268 0"/> -->
-    <!-- <origin xyz="0.032 0 0.045" rpy="0 -1.5707963268 0"/> -->
+    <!-- <origin xyz="-0.035 0 0.03" rpy="0 1.5707963268 0"/> -->
+    <origin xyz="0.032 0 0.045" rpy="0 -1.5707963268 0"/>
   </xacro:sensor_d405>
+  <xacro:include filename="$(find robotiq_2f_85_gripper_visualization)/urdf/robotiq_arg2f_85_model_macro.xacro" />
+  <xacro:robotiq_arg2f_85 prefix=""/>
+  <joint name="ur5e_gripper_link" type="fixed">
+    <origin xyz="0 0 0" rpy="0 1.5707963268 0" />
+    <parent link="flange"/>
+    <child link="robotiq_arg2f_base_link"/>
+  </joint>
 </robot>

File: robot_moveit/cam_ur5e_moveit_config/config/gazebo_ur5e_robot.urdf (robot description, URDF)
Before this commit: robot ur5e_robot, 21 links, 20 joints
Links:
- link camera_link: geometry collision box size=0.023 0.042 0.042; visual mesh filename=file:///home/fatfat/work/src/camera_models/realsense2_descr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 scale=0.001 0.001 0.001
