Commit message: [almost] cam_ur5e gripper

File: robot_models/universal_robots/ur_description/urdf/ur5e_cam.urdf.xacro (robot description, xacro)
@@ -35,5 +35,5 @@
                      align_depth="$(arg align_depth)"
                      enable_pointCloud="$(arg enable_pointCloud)">
-    <!-- <origin xyz="0 0 0" rpy="0 -1.5707963268 0"/> -->
+    <origin xyz="0 0 0" rpy="0 -1.5707963268 0"/>
     <!-- <origin xyz="0.032 0 0.045" rpy="0 -1.5707963268 0"/> -->
   </xacro:sensor_d405>

File: robot_moveit/cam_ur5e_gripper_moveit_config/config/gazebo_ur5e_robot.urdf (robot description, URDF)
Before this commit: robot ur5e_robot, 33 links, 32 joints
Links:
- link camera_link: geometry collision box size=0.023 0.042 0.042; visual mesh filename=file:///home/fatfat/work/src/camera_models/realsense2_descr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 scale=0.001 0.001 0.001
