Commit message: [tmp] gazebo moveit controller failed

File: robot_models/universal_robots/ur_description/urdf/ur5e_cam_robotiq.urdf.xacro (robot description, xacro)
@@ -68,5 +68,5 @@
   </link>
   <joint name="robotiq_coupler_joint" type="fixed">
-    <origin xyz="0 0 0.004" rpy="0 0 ${-pi/2.0}" />
+    <origin xyz="0 0 0.004" rpy="0 0 ${-M_PI/2.0}" />
     <parent link="tool0"/>
     <child link="robotiq_coupler"/>
@@ -79,5 +79,5 @@
   <!-- Attach the robotiq 85 gripper -->
   <xacro:robotiq_85_gripper prefix="" parent="robotiq_coupler" >
-    <origin xyz="0 0 0.004" rpy="0 ${-pi/2} ${pi}"/>
+    <origin xyz="0 0 0.004" rpy="0 ${-M_PI/2} ${M_PI}"/>
   </xacro:robotiq_85_gripper>
   <!-- Gazebo FT sensor plugin -->

File: robot_models/universal_robots/ur_gazebo/urdf/ur_cam_robotiq.xacro (robot description, xacro)
@@ -149,5 +149,5 @@
   </link>
   <joint name="robotiq_coupler_joint" type="fixed">
-    <origin xyz="0 0 0.004" rpy="0 0 ${-pi/2.0}" />
+    <origin xyz="0 0 0.004" rpy="0 0 ${-M_PI/2.0}" />
     <parent link="tool0"/>
     <child link="robotiq_coupler"/>
@@ -160,5 +160,5 @@
   <!-- Attach the robotiq 85 gripper -->
   <xacro:robotiq_85_gripper prefix="" parent="robotiq_coupler" >
-    <origin xyz="0 0 0.004" rpy="0 ${-pi/2} ${pi}"/>
+    <origin xyz="0 0 0.004" rpy="0 ${-M_PI/2} ${M_PI}"/>
   </xacro:robotiq_85_gripper>
   <!-- Gazebo FT sensor plugin -->
