Commit message: [ok] d405_link

File: camera_models/d405_link/urdf/d405_link.urdf (robot description, URDF)
Before this commit: robot d405_link, 1 links, 0 joints
Links:
- added link world
Joints:
- added joint cam_d405_link: type fixed, parent world, child base_link, origin xyz=0 0 0 rpy=0 0 0

Commit message: [ok] cam_ur5e_gripper

File: camera_models/d405_link/urdf/d405_link.urdf (robot description, URDF)
Before this commit: robot d405_link, 2 links, 1 joints
Links:
- removed link base_link
- removed link world
- added link connect_d405_base_link, mass 0.035381; collision mesh filename=package://d405_link/meshes/base_link.STL; visual mesh filename=package://d405_link/meshes/base_link.STL
Joints:
- removed joint cam_d405_link

File: robot_models/universal_robots/ur_description/urdf/ur5e_cam_gripper.urdf.xacro (robot description, xacro)
@@ -14,7 +14,14 @@
     Refer to 'inc/ur_macro.xacro' for more information.
   -->
+  <xacro:property name="M_PI" value="3.1415926535897931" />
+  <!--Robot UR5e-->
   <xacro:include filename="$(find ur_description)/urdf/inc/ur5e_macro.xacro"/>
   <xacro:ur5e_robot prefix="" />
-  <!--camera-->
+  <!--Connect Camera Link-->
+  <xacro:include filename="$(find d405_link)/urdf/d405_link.urdf.xacro" />
+  <xacro:connect_d405_link parent="flange">
+    <origin xyz="0.001 0 0" rpy="0 ${-M_PI/2} 0" />
+  </xacro:connect_d405_link>
+  <!--Camera D405-->
   <xacro:arg name="name"                    default="camera"/>
   <xacro:arg name="topics_ns"               default="camera"/>
@@ -24,8 +31,5 @@
   <xacro:arg name="enable_pointCloud"       default="true"/>
   <xacro:include filename="$(find realsense2_description)/urdf/_d405.urdf.xacro" />
-  <!-- <xacro:sensor_d405 parent="wrist_3_link" use_nominal_extrinsics="$(arg use_nominal_extrinsics)">
-    <origin xyz="0 0 0" rpy="0 -1.5707963268 0"/>
-  </xacro:sensor_d405> -->
-  <xacro:sensor_d405 parent="flange"
+  <xacro:sensor_d405 parent="connect_d405_base_link"
                      name="$(arg name)"
                      topics_ns="$(arg topics_ns)"
@@ -34,12 +38,12 @@
                      align_depth="$(arg align_depth)"
                      enable_pointCloud="$(arg enable_pointCloud)">
-    <!-- <origin xyz="-0.035 0 0.03" rpy="0 1.5707963268 0"/> -->
-    <origin xyz="0.032 0 0.045" rpy="0 -1.5707963268 0"/>
+    <origin xyz="-0.075 0 0.015" rpy="0 ${-M_PI*1.35} 0"/>
   </xacro:sensor_d405>
+  <!--Gripper Robotiq-2F85-->
   <xacro:include filename="$(find robotiq_2f_85_gripper_visualization)/urdf/robotiq_arg2f_85_model_macro.xacro" />
   <xacro:robotiq_arg2f_85 prefix=""/>
   <joint name="ur5e_gripper_link" type="fixed">
-    <origin xyz="0 0 0" rpy="0 1.5707963268 0" />
-    <parent link="flange"/>
+    <origin xyz="0 0 -0.01" rpy="0 ${M_PI} 0" />
+    <parent link="connect_d405_base_link"/>
     <child link="robotiq_arg2f_base_link"/>
   </joint>

File: robot_moveit/cam_ur5e_gripper_moveit_config/config/gazebo_ur5e_robot.urdf (robot description, URDF)
Before this commit: robot ur5e_robot, 32 links, 31 joints
Links:
- added link connect_d405_base_link, mass 0.035381; collision mesh filename=package://d405_link/meshes/base_link.STL; visual mesh filename=package://d405_link/meshes/base_link.STL
- link camera_link: geometry collision box size=0.023 0.042 0.042; visual mesh filename=file:///home/user/work/src/camera_models/realsense2_descrip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 scale=0.001 0.001 0.001
Joints:
- added joint connect_d405_base_link_joint: type fixed, parent flange, child connect_d405_base_link, origin xyz=0.001 0 0 rpy=0 -1.5707963267948966 0
- joint camera_joint: origin xyz=0.032 0 0.045 rpy=0 -1.5707963268 0 -> xyz=-0.075 0 0.015 rpy=0 -4.241150082346221 0; parent flange -> connect_d405_base_link
- joint ur5e_gripper_link: origin xyz=0 0 0 rpy=0 1.5707963268 0 -> xyz=0 0 -0.01 rpy=0 3.141592653589793 0; parent flange -> connect_d405_base_link
