Commit message: [ok] cam_ur5e ur5e+D405+belt

File: robot_models/universal_robots/ur_description/urdf/inc/ur_cam_macro.xacro (robot description, xacro)
@@ -319,8 +319,24 @@
     </joint>
     <!--camera-->
-    <xacro:arg name="use_nominal_extrinsics" default="true"/>
+    <!-- <xacro:arg name="use_nominal_extrinsics" default="true"/>
     <xacro:sensor_d405 parent="${prefix}wrist_3_link" use_nominal_extrinsics="$(arg use_nominal_extrinsics)">
       <origin xyz="0 0 0" rpy="0 -1.5707963268 0"/>
+    </xacro:sensor_d405> -->
+    <xacro:arg name="name"                    default="camera"/>
+    <xacro:arg name="topics_ns"               default="camera"/>
+    <xacro:arg name="use_nominal_extrinsics"  default="true"/>
+    <xacro:arg name="visualize_color"         default="true"/>
+    <xacro:arg name="align_depth"             default="true"/>
+    <xacro:arg name="enable_pointCloud"       default="true"/>
+    <!-- <xacro:include filename="$(find realsense2_description)/urdf/_d405.urdf.xacro" /> -->
+    <xacro:sensor_d405 parent="${prefix}wrist_3_link"
+                      name="$(arg name)"
+                      topics_ns="$(arg topics_ns)"
+                      use_nominal_extrinsics="$(arg use_nominal_extrinsics)"
+                      visualize_color="$(arg visualize_color)"
+                      align_depth="$(arg align_depth)"
+                      enable_pointCloud="$(arg enable_pointCloud)">
+      <origin xyz="0 0 0" rpy="0 -1.5707963268 0"/>
     </xacro:sensor_d405>
-  </xacro:macro>
+    </xacro:macro>
 </robot>

File: robot_models/universal_robots/ur_gazebo/urdf/ur.xacro (robot description, xacro)
@@ -29,5 +29,5 @@
   <xacro:arg name="physical_params" default=""/>
   <xacro:arg name="kinematics_params" default=""/>
-  <xacro:arg name="visual_params" default=""/>
+    <xacro:arg name="visual_params" default=""/>
   <!--
     legal values:

File: robot_models/universal_robots/ur_gazebo/urdf/ur_cam.xacro (robot description, xacro)
@@ -1,7 +1,29 @@
 <?xml version="1.0"?>
 <robot xmlns:xacro="http://wiki.ros.org/xacro" name="$(arg robot_model)_robot">
-   <!-- import main macro -->
-   <xacro:include filename="$(find ur_description)/urdf/inc/ur_cam_macro.xacro"/>
-   <!-- parameters -->
+  <!--
+    This is a top-level xacro instantiating the Gazebo-specific version of the
+    'ur_robot' macro (ie: 'ur_robot_gazebo') and passing it values for all its
+    required arguments.
+    This file should be considered the Gazebo-specific variant of the file
+    with the same name in the ur_description package. It accepts the same
+    arguments, but instead of configuring everything for a real robot, will
+    generate a Gazebo-compatible URDF with a ros_control hardware_interface
+    attached to it.
+    Only use this top-level xacro if you plan on spawning the robot in Gazebo
+    'by itself', without any gripper or any other geometry attached.
+    If you need to attach an end-effector, camera or need to integrate the
+    robot into a larger workcell and want to spawn that as a single entity in
+    Gazebo, DO NOT EDIT THIS FILE.
+    Instead: create a new top-level xacro, give it a proper name, include the
+    required '.xacro' files, instantiate the models (ie: call the macros) and
+    connect everything by adding the appropriate joints.
+  -->
+  <!--
+    Import main macro.
+    NOTE: this imports the Gazebo-wrapper main macro, NOT the regular
+          xacro macro (which is hosted by ur_description).
+  -->
+  <xacro:include filename="$(find ur_gazebo)/urdf/ur_cam_macro.xacro"/>
+  <!--Declare arguments -->
    <xacro:arg name="joint_limit_params" default=""/>
    <xacro:arg name="kinematics_params" default=""/>
@@ -12,11 +34,13 @@
          - hardware_interface/VelocityJointInterface
          - hardware_interface/EffortJointInterface
-   -->
-   <xacro:arg name="transmission_hw_interface" default="hardware_interface/PositionJointInterface"/>
+    NOTE: this value must correspond to the controller configured in the
+          controller .yaml files in the 'config' directory.
+  -->
+   <xacro:arg name="transmission_hw_interface" default="hardware_interface/EffortJointInterface"/>
    <xacro:arg name="safety_limits" default="false"/>
    <xacro:arg name="safety_pos_margin" default="0.15"/>
    <xacro:arg name="safety_k_position" default="20"/>
-   <!-- arm -->
-   <xacro:ur_robot
+   <!-- Instantiate the Gazebo robot and pass it all the required arguments. -->
+   <xacro:ur_robot_gazebo
      prefix=""
      joint_limits_parameters_file="$(arg joint_limit_params)"
@@ -27,4 +51,33 @@
      safety_limits="$(arg safety_limits)"
      safety_pos_margin="$(arg safety_pos_margin)"
-     safety_k_position="$(arg safety_k_position)"/>
+     safety_k_position="$(arg safety_k_position)"
+     />
+  <!--
+    Attach the Gazebo model to Gazebo's world frame.
+    Note: if you're looking to integrate a UR into a larger scene and need
+    to add EEFs or other parts, DO NOT change this file or the 'world' link
+    here. Create a NEW xacro instead and decide whether you need to add
+    a 'world' link there.
+  -->
+  <link name="world"/>
+  <joint name="world_joint" type="fixed">
+    <parent link="world"/>
+    <child link="base_link"/>
+    <origin xyz="0 0 0" rpy="0 0 0"/>
+  </joint>
+  <link name="tool0_controller"/>
+  <joint name="tool_controller_fake_joint" type="fixed">
+    <parent link="tool0"/>
+    <child link="tool0_controller"/>
+    <origin xyz="0 0 0" rpy="0 0 0"/>
+  </joint>
+  <xacro:include filename="$(find belt12mm_description)/urdf/belt12mm.xacro"/>
+  <xacro:belt12mm parent="base_link" prefix="belt12mm_">
+    <origin xyz="0.0 0.0 0.0" rpy="0.0 0.0 0.0"/>
+  </xacro:belt12mm>
+  <joint name="belt12mm_joint" type="fixed">
+          <parent link="base_link"/>
+          <child link="belt12mm_base_link"/>
+          <origin xyz="0.5 0.0 0" rpy="1.57 0 1.57"/>
+  </joint>
 </robot>

File: robot_models/universal_robots/ur_gazebo/urdf/ur_cam_macro.xacro (robot description, xacro)
@@ -2,8 +2,5 @@
 <robot xmlns:xacro="http://wiki.ros.org/xacro">
   <!--
-    Main xacro macro definition of the "Gazebo robot" model.
-    This wraps the model of the real robot and adds all elements and parameters
-    required by Gazebo.
-    It also adds the gazebo_ros_control plugin.
+    Base UR robot series xacro macro.
     NOTE: this is NOT a URDF. It cannot directly be loaded by consumers
     expecting a flattened '.urdf' file. See the top-level '.xacro' for that
@@ -11,24 +8,42 @@
     For use in '.launch' files: use one of the 'load_urX.launch' convenience
     launch files.
-    NOTE: this Gazebo model makes use of the same set of parameter files as the
-    main xacro macro (in ur_description). It is therefor possible to use the
-    kinematic calibration exported from a REAL UR robot. Please refer to the
-    ur_macro.xacro in ur_description for more information about this.
+    This file models the base kinematic chain of a UR robot, which then gets
+    parameterised by various configuration files to convert it into a UR3(e),
+    UR5(e), UR10(e), UR16e, UR20 or UR30.
+    NOTE: the default kinematic parameters (ie: link lengths, frame locations,
+    offets, etc) do not correspond to any particular robot. They are defaults
+    only. There WILL be non-zero offsets between the Forward Kinematics results
+    in TF (ie: robot_state_publisher) and the values reported by the Teach
+    Pendant.
+    For accurate (and robot-specific) transforms, the 'kinematics_parameters_file'
+    parameter MUST point to a .yaml file containing the appropriate values for
+    the targetted robot.
+    If using the UniversalRobots/Universal_Robots_ROS_Driver, follow the steps
+    described in the readme of that repository to extract the kinematic
+    calibration from the controller and generate the required .yaml file.
     Main author of the migration to yaml configs: Ludovic Delval.
     Contributors to previous versions (in no particular order):
      - Felix Messmer
      - Kelsey Hawkins
+     - Wim Meeussen
      - Shaun Edwards
-     - Alexander Bubeck
      - Nadia Hammoudeh Garcia
+     - Dave Hershberger
      - G. vd. Hoorn
-     - Dave Niewinski
-     - Andy Zelenak
+     - Philip Long
+     - Dave Coleman
      - Miguel Prada
      - Mathias Luedtke
-     - Hans-Joachim Krauch
+     - Marcel Schnirring
+     - Felix von Drigalski
      - Felix Exner
+     - Jimmy Da Silva
+     - Ajit Krisshna N L
+     - Muhammad Asif Rana
   -->
-  <!-- Definition of the main macro -->
+  <!-- <xacro:include filename="$(find ur_description)/urdf/inc/ur_transmissions.xacro" />
+  <xacro:include filename="$(find ur_description)/urdf/inc/ur_common.xacro" /> -->
+  <!--camera-->
+  <!-- <xacro:include filename="$(find realsense2_description)/urdf/_d405.urdf.xacro" /> -->
   <xacro:macro name="ur_robot_gazebo" params="
     prefix
@@ -48,5 +63,5 @@
       the definitions for the real robot.
     -->
-    <xacro:include filename="$(find ur_description)/urdf/inc/ur_macro.xacro"/>
+    <xacro:include filename="$(find ur_description)/urdf/inc/ur_cam_macro.xacro"/>
     <!-- Instantiate model for the REAL robot. -->
     <xacro:ur_robot
@@ -93,4 +108,25 @@
       </plugin>
     </gazebo>
-  </xacro:macro>
+    <!--camera-->
+    <!-- <xacro:arg name="use_nominal_extrinsics" default="true"/>
+    <xacro:sensor_d405 parent="${prefix}wrist_3_link" use_nominal_extrinsics="$(arg use_nominal_extrinsics)">
+      <origin xyz="0 0 0" rpy="0 -1.5707963268 0"/>
+    </xacro:sensor_d405> -->
+    <!-- <xacro:arg name="name"                    default="camera"/>
+    <xacro:arg name="topics_ns"               default="camera"/>
+    <xacro:arg name="use_nominal_extrinsics"  default="true"/>
+    <xacro:arg name="visualize_color"         default="true"/>
+    <xacro:arg name="align_depth"             default="true"/>
+    <xacro:arg name="enable_pointCloud"       default="true"/> -->
+    <!-- <xacro:include filename="$(find realsense2_description)/urdf/_d405.urdf.xacro" /> -->
+    <!-- <xacro:sensor_d405 parent="${prefix}wrist_3_link"
+                      name="$(arg name)"
+                      topics_ns="$(arg topics_ns)"
+                      use_nominal_extrinsics="$(arg use_nominal_extrinsics)"
+                      visualize_color="$(arg visualize_color)"
+                      align_depth="$(arg align_depth)"
+                      enable_pointCloud="$(arg enable_pointCloud)">
+      <origin xyz="0 0 0" rpy="0 -1.5707963268 0"/>
+    </xacro:sensor_d405> -->
+    </xacro:macro>
 </robot>

Commit message: [almost] cam_ur5e_gripper

File: robot_models/universal_robots/ur_description/urdf/inc/ur_cam_macro.xacro (robot description, xacro)
@@ -44,6 +44,6 @@
   <xacro:include filename="$(find ur_description)/urdf/inc/ur_transmissions.xacro" />
   <xacro:include filename="$(find ur_description)/urdf/inc/ur_common.xacro" />
-  <!--camera-->
-  <xacro:include filename="$(find realsense2_description)/urdf/_d405.urdf.xacro" />
+  <!--Camera-->
+  <!-- <xacro:include filename="$(find realsense2_description)/urdf/_d405.urdf.xacro" /> -->
   <xacro:macro name="ur_robot" params="
     prefix
@@ -323,12 +323,12 @@
       <origin xyz="0 0 0" rpy="0 -1.5707963268 0"/>
     </xacro:sensor_d405> -->
-    <xacro:arg name="name"                    default="camera"/>
+    <!-- <xacro:arg name="name"                    default="camera"/>
     <xacro:arg name="topics_ns"               default="camera"/>
     <xacro:arg name="use_nominal_extrinsics"  default="true"/>
     <xacro:arg name="visualize_color"         default="true"/>
     <xacro:arg name="align_depth"             default="true"/>
-    <xacro:arg name="enable_pointCloud"       default="true"/>
+    <xacro:arg name="enable_pointCloud"       default="true"/> -->
     <!-- <xacro:include filename="$(find realsense2_description)/urdf/_d405.urdf.xacro" /> -->
-    <xacro:sensor_d405 parent="${prefix}wrist_3_link"
+    <!-- <xacro:sensor_d405 parent="${prefix}wrist_3_link"
                       name="$(arg name)"
                       topics_ns="$(arg topics_ns)"
@@ -338,5 +338,22 @@
                       enable_pointCloud="$(arg enable_pointCloud)">
       <origin xyz="0 0 0" rpy="0 -1.5707963268 0"/>
-    </xacro:sensor_d405>
+    </xacro:sensor_d405> -->
+    <!--Camera D405-->
+    <!-- <xacro:arg name="name"                    default="camera"/>
+    <xacro:arg name="topics_ns"               default="camera"/>
+    <xacro:arg name="use_nominal_extrinsics"  default="true"/>
+    <xacro:arg name="visualize_color"         default="true"/>
+    <xacro:arg name="align_depth"             default="true"/>
+    <xacro:arg name="enable_pointCloud"       default="true"/> -->
+    <!-- <xacro:include filename="$(find realsense2_description)/urdf/_d405.urdf.xacro" /> -->
+    <!-- <xacro:sensor_d405 parent="connect_d405_base_link"
+                      name="$(arg name)"
+                      topics_ns="$(arg topics_ns)"
+                      use_nominal_extrinsics="$(arg use_nominal_extrinsics)"
+                      visualize_color="$(arg visualize_color)"
+                      align_depth="$(arg align_depth)"
+                      enable_pointCloud="$(arg enable_pointCloud)">
+      <origin xyz="-0.075 0 0.015" rpy="0 ${-M_PI*1.35} 0"/>
+    </xacro:sensor_d405> -->
     </xacro:macro>
 </robot>

File: robot_models/universal_robots/ur_gazebo/urdf/ur_cam.xacro (robot description, xacro)
@@ -72,4 +72,5 @@
     <origin xyz="0 0 0" rpy="0 0 0"/>
   </joint>
+  <!--PU Belt-->
   <xacro:include filename="$(find belt12mm_description)/urdf/belt12mm.xacro"/>
   <xacro:belt12mm parent="base_link" prefix="belt12mm_">
@@ -81,3 +82,21 @@
           <origin xyz="0.5 0.0 0" rpy="1.57 0 1.57"/>
   </joint>
+  <!--Camera D405-->
+  <xacro:arg name="name"                    default="camera"/>
+  <xacro:arg name="topics_ns"               default="camera"/>
+  <xacro:arg name="use_nominal_extrinsics"  default="true"/>
+  <xacro:arg name="visualize_color"         default="true"/>
+  <xacro:arg name="align_depth"             default="true"/>
+  <xacro:arg name="enable_pointCloud"       default="true"/>
+  <xacro:include filename="$(find realsense2_description)/urdf/_d405.urdf.xacro" />
+  <!-- <xacro:sensor_d405 parent="${prefix}wrist_3_link"  -->
+  <xacro:sensor_d405 parent="wrist_3_link"
+                    name="$(arg name)"
+                    topics_ns="$(arg topics_ns)"
+                    use_nominal_extrinsics="$(arg use_nominal_extrinsics)"
+                    visualize_color="$(arg visualize_color)"
+                    align_depth="$(arg align_depth)"
+                    enable_pointCloud="$(arg enable_pointCloud)">
+    <origin xyz="0 0 0" rpy="0 -1.5707963268 0"/>
+  </xacro:sensor_d405>
 </robot>

File: robot_models/universal_robots/ur_gazebo/urdf/ur_cam_gripper.xacro (robot description, xacro)
@@ -97,4 +97,21 @@
     <origin xyz="0.001 0 0" rpy="0 ${-M_PI/2} 0" />
   </xacro:connect_d405_link>
+  <!--Camera D405-->
+  <xacro:arg name="name"                    default="camera"/>
+  <xacro:arg name="topics_ns"               default="camera"/>
+  <xacro:arg name="use_nominal_extrinsics"  default="true"/>
+  <xacro:arg name="visualize_color"         default="true"/>
+  <xacro:arg name="align_depth"             default="true"/>
+  <xacro:arg name="enable_pointCloud"       default="true"/>
+  <xacro:include filename="$(find realsense2_description)/urdf/_d405.urdf.xacro" />
+  <xacro:sensor_d405 parent="connect_d405_base_link"
+                     name="$(arg name)"
+                     topics_ns="$(arg topics_ns)"
+                     use_nominal_extrinsics="$(arg use_nominal_extrinsics)"
+                     visualize_color="$(arg visualize_color)"
+                     align_depth="$(arg align_depth)"
+                     enable_pointCloud="$(arg enable_pointCloud)">
+    <origin xyz="-0.075 0 0.015" rpy="0 ${-M_PI*1.35} 0"/>
+  </xacro:sensor_d405>
   <!--Gripper Robotiq-2F85-->
   <xacro:include filename="$(find robotiq_2f_85_gripper_visualization)/urdf/robotiq_arg2f_85_model_macro.xacro" />
